File: pcb/pcb.kicad_sch (KiCad schematic)
At the start: 57 parts, among them J1 N!N, J2 Conn_01x02_Socket, J4 Display_nice-view, J8 Conn_01x12_Socket, J9 Conn_01x12_Socket, SW10 Switch, SW11 Switch, SW12 Switch, SW13 Switch, SW14 Switch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

Commit message: converting duet to standard x and min y spacing, along with strong pinky stagger, WIP
Parts:
- SW10, SW11, SW12, SW13, SW14, SW15, SW18, SW19, SW3, SW4, SW5, SW6, SW7, SW8, SW9: footprint zzkeeb:Switch_ChocV1-hotswap-reversible -> fingerpunch:Switch_ChocV1-hotswap-minY-reversible
Changed lines of the file:
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@@
       (effects (font (size 1.27 1.27)) hide)
     )
-    (property "Footprint" "zzkeeb:Switch_ChocV1-hotswap-reversible" (at 38.1 133.35 0)
+    (property "Footprint" "fingerpunch:Switch_ChocV1-hotswap-minY-reversible" (at 38.1 133.35 0)
       (effects (font (size 1.27 1.27)) hide)
     )
@@
       (effects (font (size 1.27 1.27)) hide)
     )
-    (property "Footprint" "zzkeeb:Switch_ChocV1-hotswap-reversible" (at 91.44 92.71 0)
+    (property "Footprint" "fingerpunch:Switch_ChocV1-hotswap-minY-reversible" (at 91.44 92.71 0)
       (effects (font (size 1.27 1.27)) hide)
     )
@@
       (effects (font (size 1.27 1.27)) hide)
     )
-    (property "Footprint" "zzkeeb:Switch_ChocV1-hotswap-reversible" (at 73.66 113.03 0)
+    (property "Footprint" "fingerpunch:Switch_ChocV1-hotswap-minY-reversible" (at 73.66 113.03 0)
       (effects (font (size 1.27 1.27)) hide)
     )
@@
       (effects (font (size 1.27 1.27)) hide)
     )
-    (property "Footprint" "zzkeeb:Switch_ChocV1-hotswap-reversible" (at 91.44 153.67 0)
+    (property "Footprint" "fingerpunch:Switch_ChocV1-hotswap-minY-reversible" (at 91.44 153.67 0)
       (effects (font (size 1.27 1.27)) hide)
     )
@@
       (effects (font (size 1.27 1.27)) hide)
     )
-    (property "Footprint" "zzkeeb:Switch_ChocV1-hotswap-reversible" (at 109.22 133.35 0)
+    (property "Footprint" "fingerpunch:Switch_ChocV1-hotswap-minY-reversible" (at 109.22 133.35 0)
       (effects (font (size 1.27 1.27)) hide)
     )
@@
       (effects (font (size 1.27 1.27)) hide)
     )
-    (property "Footprint" "zzkeeb:Switch_ChocV1-hotswap-reversible" (at 109.22 153.67 0)
+    (property "Footprint" "fingerpunch:Switch_ChocV1-hotswap-minY-reversible" (at 109.22 153.67 0)
       (effects (font (size 1.27 1.27)) hide)
     )
@@
       (effects (font (size 1.27 1.27)) hide)
     )
-    (property "Footprint" "zzkeeb:Switch_ChocV1-hotswap-reversible" (at 38.1 153.67 0)
+    (property "Footprint" "fingerpunch:Switch_ChocV1-hotswap-minY-reversible" (at 38.1 153.67 0)
       (effects (font (size 1.27 1.27)) hide)
     )
@@
       (effects (font (size 1.27 1.27)) hide)
     )
-    (property "Footprint" "zzkeeb:Switch_ChocV1-hotswap-reversible" (at 73.66 153.67 0)
+    (property "Footprint" "fingerpunch:Switch_ChocV1-hotswap-minY-reversible" (at 73.66 153.67 0)
       (effects (font (size 1.27 1.27)) hide)
     )
@@
       (effects (font (size 1.27 1.27)) hide)
     )
-    (property "Footprint" "zzkeeb:Switch_ChocV1-hotswap-reversible" (at 73.66 92.71 0)
+    (property "Footprint" "fingerpunch:Switch_ChocV1-hotswap-minY-reversible" (at 73.66 92.71 0)
       (effects (font (size 1.27 1.27)) hide)
     )
@@
       (effects (font (size 1.27 1.27)) hide)
     )
-    (property "Footprint" "zzkeeb:Switch_ChocV1-hotswap-reversible" (at 73.66 133.35 0)
+    (property "Footprint" "fingerpunch:Switch_ChocV1-hotswap-minY-reversible" (at 73.66 133.35 0)
       (effects (font (size 1.27 1.27)) hide)
     )
@@
       (effects (font (size 1.27 1.27)) hide)
     )
-    (property "Footprint" "zzkeeb:Switch_ChocV1-hotswap-reversible" (at 38.1 113.03 0)
+    (property "Footprint" "fingerpunch:Switch_ChocV1-hotswap-minY-reversible" (at 38.1 113.03 0)
       (effects (font (size 1.27 1.27)) hide)
     )
@@
       (effects (font (size 1.27 1.27)) hide)
     )
-    (property "Footprint" "zzkeeb:Switch_ChocV1-hotswap-reversible" (at 38.1 92.71 0)
+    (property "Footprint" "fingerpunch:Switch_ChocV1-hotswap-minY-reversible" (at 38.1 92.71 0)
       (effects (font (size 1.27 1.27)) hide)
     )
@@
       (effects (font (size 1.27 1.27)) hide)
     )
-    (property "Footprint" "zzkeeb:Switch_ChocV1-hotswap-reversible" (at 109.22 113.03 0)
+    (property "Footprint" "fingerpunch:Switch_ChocV1-hotswap-minY-reversible" (at 109.22 113.03 0)
       (effects (font (size 1.27 1.27)) hide)
     )
@@
       (effects (font (size 1.27 1.27)) hide)
     )
-    (property "Footprint" "zzkeeb:Switch_ChocV1-hotswap-reversible" (at 91.44 113.03 0)
+    (property "Footprint" "fingerpunch:Switch_ChocV1-hotswap-minY-reversible" (at 91.44 113.03 0)
       (effects (font (size 1.27 1.27)) hide)
     )
@@
       (effects (font (size 1.27 1.27)) hide)
     )
-    (property "Footprint" "zzkeeb:Switch_ChocV1-hotswap-reversible" (at 55.88 113.03 0)
+    (property "Footprint" "fingerpunch:Switch_ChocV1-hotswap-minY-reversible" (at 55.88 113.03 0)
       (effects (font (size 1.27 1.27)) hide)
     )
@@
       (effects (font (size 1.27 1.27)) hide)
     )
-    (property "Footprint" "zzkeeb:Switch_ChocV1-hotswap-reversible" (at 55.88 133.35 0)
+    (property "Footprint" "fingerpunch:Switch_ChocV1-hotswap-minY-reversible" (at 55.88 133.35 0)
       (effects (font (size 1.27 1.27)) hide)
     )
@@
       (effects (font (size 1.27 1.27)) hide)
     )
-    (property "Footprint" "zzkeeb:Switch_ChocV1-hotswap-reversible" (at 55.88 92.71 0)
+    (property "Footprint" "fingerpunch:Switch_ChocV1-hotswap-minY-reversible" (at 55.88 92.71 0)
       (effects (font (size 1.27 1.27)) hide)
     )
@@
       (effects (font (size 1.27 1.27)) hide)
     )
-    (property "Footprint" "zzkeeb:Switch_ChocV1-hotswap-reversible" (at 109.22 92.71 0)
+    (property "Footprint" "fingerpunch:Switch_ChocV1-hotswap-minY-reversible" (at 109.22 92.71 0)
       (effects (font (size 1.27 1.27)) hide)
     )
@@
       (effects (font (size 1.27 1.27)) hide)
     )
-    (property "Footprint" "zzkeeb:Switch_ChocV1-hotswap-reversible" (at 55.88 153.67 0)
+    (property "Footprint" "fingerpunch:Switch_ChocV1-hotswap-minY-reversible" (at 55.88 153.67 0)
       (effects (font (size 1.27 1.27)) hide)
     )
@@
       (effects (font (size 1.27 1.27)) hide)
     )
-    (property "Footprint" "zzkeeb:Switch_ChocV1-hotswap-reversible" (at 91.44 133.35 0)
-      (effects (font (size 1.27 1.27)) hide)
-    )
+    (property "Footprint" "fingerpunch:Switch_ChocV1-hotswap-minY-reversible" (at 91.44 133.35 0)
+      (effects (font (size 1.27 1.27)) hide)
+    )
